File: ESP32-wroover-adapter.kicad_pcb (KiCad board)
At the start: 2 copper layers, 33.7 x 53.3 mm, 20 parts, among them J1 USB_OTG, J2 Screw_Terminal_01x03, J3 Screw_Terminal_01x03, J4 Screw_Terminal_01x03, J5 Screw_Terminal_01x03, J6 Conn_01x20, J7 Conn_01x07, J8 Screw_Terminal_01x02, J9 Conn_01x04, Q1 Q_NPN_BCE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

Commit message: update
Parts:
- added C1: C, Capacitors_SMD:C_0603, F.Cu at (99.7, 83.2)
- added C2: C, Capacitors_SMD:C_0603, F.Cu at (102.9, 70.5)
- added C3: C, Capacitors_SMD:C_0603, F.Cu at (102.9, 75.6)
- added C4: C, Capacitors_SMD:C_0603, F.Cu at (94.0, 87.0)
- added C5: C, Capacitors_SMD:C_0603, F.Cu at (104.8, 79.4)
- added C6: C, Capacitors_SMD:C_0603, F.Cu at (102.9, 86.4)
- added C7: C, Capacitors_SMD:C_0603, F.Cu at (88.9, 94.6)
- added D2: LED, LEDs:LED_0603, F.Cu at (102.9, 68.6)
- added R10: R, Resistors_SMD:R_0603, F.Cu at (97.8, 94.6)
- added R11: R, Resistors_SMD:R_0603, F.Cu at (93.3, 94.6)
- added R3: R, Resistors_SMD:R_0603, F.Cu at (64.1, 68.6)
- added R4: R, Resistors_SMD:R_0603, F.Cu at (64.1, 71.8)
- added R5: R, Resistors_SMD:R_0603, F.Cu at (91.4, 83.2)
- added R6: R, Resistors_SMD:R_0603, F.Cu at (97.8, 71.1)
- added R7: R, Resistors_SMD:R_0603, F.Cu at (97.8, 76.8)
- added R8: R, Resistors_SMD:R_0603, F.Cu at (106.0, 94.0)
- added R9: R, Resistors_SMD:R_0603, F.Cu at (101.6, 94.6)
- R1, R2: footprint Resistors_SMD:R_0805 -> Resistors_SMD:R_0603
- moved D1 31.7 mm to (57.8, 70.5)
- moved J9 12.1 mm to (73.7, 66.7), turned to 180 degrees
- moved U3 7.65 mm to (56.5, 59.7)
- moved U1 7.01 mm to (54.0, 69.8)
- moved R2 4.02 mm to (70.5, 85.7)
- moved U2 3.18 mm to (56.5, 83.2)
- moved Q2 2.62 mm to (64.8, 76.2)
- moved Q3 2.01 mm to (64.8, 85.1)
- moved Q1 1.27 mm to (56.5, 75.6)

Commit message: update
Parts:
- added J10: Micro_SD_Card, digikey-footprints:DM3D-SF, F.Cu at (80.6, 65.4)
- J7: footprint Pin_Headers:Pin_Header_Angled_1x07_Pitch2.54mm -> Pin_Headers:Pin_Header_Straight_1x07_Pitch2.54mm
- moved J8 60.3 mm to (19.7, 71.8)
- moved J3 42.7 mm to (37.5, 60.3)
- moved J9 7.43 mm to (66.7, 69.2)
- moved R3 4.84 mm to (59.7, 66.7)
