File: ESP32-wroover-adapter.sch (KiCad schematic (older format))
At the start: 1 part, among them U1 ESP32-WROVER

Commit message: update
Parts:
- added Q1, Q2: Q_NPN_BCE, symbol Q_NPN_BCE
- added R? (x2): R, symbol R
- added U?: CP2104, Housings_DFN_QFN:QFN-24-1EP_4x4mm_Pitch0.5mm, symbol CP2104
- added U?: ap2112, symbol ap2112
Connections:
- net labels removed: GND
- wire segments 63 -> 4
Other:
- moved on the sheet: U1

Commit message: update
Parts:
- added D1: D_Schottky, Diodes_SMD:D_1206, symbol D_Schottky
- added J1: USB_OTG, Connectors_USB:USB_Micro-B_Molex-105017-0001, symbol USB_OTG
- added J2, J3, J4, J5: Screw_Terminal_01x03, TerminalBlocks_Phoenix:TerminalBlock_Phoenix_MPT-2.54mm_3pol, symbol Screw_Terminal_01x03
- added J6: Conn_01x20, Pin_Headers:Pin_Header_Straight_1x20_Pitch2.54mm, symbol Conn_01x20
- added J7: Conn_01x07, Pin_Headers:Pin_Header_Angled_1x07_Pitch2.54mm, symbol Conn_01x07
- added J8: Screw_Terminal_01x02, TerminalBlocks_Phoenix:TerminalBlock_Phoenix_MPT-2.54mm_2pol, symbol Screw_Terminal_01x02
- added J?: Conn_01x04, symbol Conn_01x04
- added Q3: Q_PMOS_DGS, digikey-footprints:SOT-23-3, symbol Q_PMOS_DGS
- added SW1: SW_Push, Buttons_Switches_SMD:SW_SPST_EVQP2, symbol SW_Push
- added U3: BME280, hog32:BME280, symbol BME280
- Q1, Q2: footprint (none) -> digikey-footprints:SOT-23-3
- R1, R2: renamed from R?; footprint (none) -> Resistors_SMD:R_0805
- U2: renamed from U?; footprint (none) -> TO_SOT_Packages_SMD:TSOT-23-5
- gave numbers to parts that had none: 1
Other:
- moved on the sheet: U2, U4
Changed lines of the file:
@@
 LIBS:ap2112
 LIBS:hog32
+LIBS:switches
+LIBS:nqbit
 LIBS:ESP32-wroover-adapter-cache
 EELAYER 25 0
@@
 F 0 "Q1" H 5350 4700 50  0000 L CNN
 F 1 "Q_NPN_BCE" H 5350 4600 50  0000 L CNN
-F 2 "" H 5350 4750 50  0001 C CNN
+F 2 "digikey-footprints:SOT-23-3" H 5350 4750 50  0001 C CNN
 F 3 "" H 5150 4650 50  0001 C CNN
 	1    5150 4650
@@
 F 0 "Q2" H 5350 5350 50  0000 L CNN
 F 1 "Q_NPN_BCE" H 5350 5250 50  0000 L CNN
-F 2 "" H 5350 5400 50  0001 C CNN
+F 2 "digikey-footprints:SOT-23-3" H 5350 5400 50  0001 C CNN
 F 3 "" H 5150 5300 50  0001 C CNN
 	1    5150 5300
@@
 $EndComp
 $Comp
-L R R?
+L R R1
 U 1 1 5B2AE0EE
 P 4800 4650
-F 0 "R?" V 4880 4650 50  0000 C CNN
+F 0 "R1" V 4880 4650 50  0000 C CNN
 F 1 "R" V 4800 4650 50  0000 C CNN
-F 2 "" V 4730 4650 50  0001 C CNN
+F 2 "Resistors_SMD:R_0805" V 4730 4650 50  0001 C CNN
 F 3 "" H 4800 4650 50  0001 C CNN
 	1    4800 4650
@@
 $EndComp
 $Comp
-L R R?
+L R R2
 U 1 1 5B2AE153
 P 4800 5300
-F 0 "R?" V 4880 5300 50  0000 C CNN
+F 0 "R2" V 4880 5300 50  0000 C CNN
 F 1 "R" V 4800 5300 50  0000 C CNN
-F 2 "" V 4730 5300 50  0001 C CNN
+F 2 "Resistors_SMD:R_0805" V 4730 5300 50  0001 C CNN
 F 3 "" H 4800 5300 50  0001 C CNN
 	1    4800 5300
@@
 $EndComp
 $Comp
-L CP2104 U?
+L CP2104 U4
 U 1 1 5B2AE1DD
-P 9500 1850
-F 0 "U?" H 9200 2775 50  0000 R CNN
-F 1 "CP2104" H 9200 2700 50  0000 R CNN
-F 2 "Housings_DFN_QFN:QFN-24-1EP_4x4mm_Pitch0.5mm" H 9650 900 50  0001 L CNN
-F 3 "" H 8950 3100 50  0001 C CNN
-	1    9500 1850
-	1    0    0    -1
-$EndComp
-$Comp
-L ap2112 U?
+P 9150 2200
+F 0 "U4" H 8850 3125 50  0000 R CNN
+F 1 "CP2104" H 8850 3050 50  0000 R CNN
+F 2 "Housings_DFN_QFN:QFN-24-1EP_4x4mm_Pitch0.5mm" H 9300 1250 50  0001 L CNN
+F 3 "" H 8600 3450 50  0001 C CNN
+	1    9150 2200
+	1    0    0    -1
+$EndComp
+$Comp
+L ap2112 U2
 U 1 1 5B2AE6D6
-P 2350 1650
-F 0 "U?" H 2350 1300 60  0000 C CNN
-F 1 "ap2112" H 2350 2000 60  0000 C CNN
-F 2 "" H 2500 1650 60  0001 C CNN
-F 3 "" H 2500 1650 60  0001 C CNN
-	1    2350 1650
-	1    0    0    -1
-$EndComp
+P 3000 1500
+F 0 "U2" H 3000 1150 60  0000 C CNN
+F 1 "ap2112" H 3000 1850 60  0000 C CNN
+F 2 "TO_SOT_Packages_SMD:TSOT-23-5" H 3150 1500 60  0001 C CNN
+F 3 "" H 3150 1500 60  0001 C CNN
+	1    3000 1500
+	1    0    0    -1
+$EndComp
+$Comp
+L BME280 U3
+U 1 1 5B2BC03D
+P 5950 1550
+F 0 "U3" H 5950 2050 60  0000 C CNN
+F 1 "BME280" H 5950 1200 60  0000 C CNN
+F 2 "hog32:BME280" H 5950 1550 60  0001 C CNN
+F 3 "" H 5950 1550 60  0001 C CNN
+	1    5950 1550
+	1    0    0    -1
+$EndComp
+$Comp
+L USB_OTG J1
+U 1 1 5B2BC711
+P 5150 3150
+F 0 "J1" H 4950 3600 50  0000 L CNN
+F 1 "USB_OTG" H 4950 3500 50  0000 L CNN
+F 2 "Connectors_USB:USB_Micro-B_Molex-105017-0001" H 5300 3100 50  0001 C CNN
+F 3 "" H 5300 3100 50  0001 C CNN
+	1    5150 3150
+	1    0    0    -1
+$EndComp
+$Comp
+L D_Schottky D1
+U 1 1 5B2BCB19
+P 1350 2050
+F 0 "D1" H 1350 2150 50  0000 C CNN
+F 1 "D_Schottky" H 1350 1950 50  0000 C CNN
+F 2 "Diodes_SMD:D_1206" H 1350 2050 50  0001 C CNN
+F 3 "" H 1350 2050 50  0001 C CNN
+	1    1350 2050
+	-1   0    0    1
+$EndComp
+$Comp
+L Q_PMOS_DGS Q3
+U 1 1 5B2BCD13
+P 1350 1200
+F 0 "Q3" H 1550 1250 50  0000 L CNN
+F 1 "Q_PMOS_DGS" H 1550 1150 50  0000 L CNN
+F 2 "digikey-footprints:SOT-23-3" H 1550 1300 50  0001 C CNN
+F 3 "" H 1350 1200 50  0001 C CNN
+	1    1350 1200
+	1    0    0    -1
+$EndComp
+$Comp
+L SW_Push SW1
+U 1 1 5B2BCF96
+P 4100 1400
+F 0 "SW1" H 4150 1500 50  0000 L CNN
+F 1 "SW_Push" H 4100 1340 50  0000 C CNN
+F 2 "Buttons_Switches_SMD:SW_SPST_EVQP2" H 4100 1600 50  0001 C CNN
+F 3 "" H 4100 1600 50  0001 C CNN
+	1    4100 1400
+	0    1    1    0
+$EndComp
+$Comp
+L Screw_Terminal_01x03 J2
+U 1 1 5B2BE424
+P 6850 2800
+F 0 "J2" H 6850 3000 50  0000 C CNN
+F 1 "Screw_Terminal_01x03" H 6850 2600 50  0000 C CNN
+F 2 "TerminalBlocks_Phoenix:TerminalBlock_Phoenix_MPT-2.54mm_3pol" H 6850 2800 50  0001 C CNN
+F 3 "" H 6850 2800 50  0001 C CNN
+	1    6850 2800
+	1    0    0    -1
+$EndComp
+$Comp
+L Screw_Terminal_01x03 J3
+U 1 1 5B2BE4D6
+P 6850 3400
+F 0 "J3" H 6850 3600 50  0000 C CNN
+F 1 "Screw_Terminal_01x03" H 6850 3200 50  0000 C CNN
+F 2 "TerminalBlocks_Phoenix:TerminalBlock_Phoenix_MPT-2.54mm_3pol" H 6850 3400 50  0001 C CNN
+F 3 "" H 6850 3400 50  0001 C CNN
+	1    6850 3400
+	1    0    0    -1
+$EndComp
+$Comp
+L Screw_Terminal_01x03 J4
+U 1 1 5B2BE530
+P 6850 3950
+F 0 "J4" H 6850 4150 50  0000 C CNN
+F 1 "Screw_Terminal_01x03" H 6850 3750 50  0000 C CNN
+F 2 "TerminalBlocks_Phoenix:TerminalBlock_Phoenix_MPT-2.54mm_3pol" H 6850 3950 50  0001 C CNN
+F 3 "" H 6850 3950 50  0001 C CNN
+	1    6850 3950
+	1    0    0    -1
+$EndComp
+$Comp
+L Screw_Terminal_01x03 J5
+U 1 1 5B2BE57F
+P 6850 4750
+F 0 "J5" H 6850 4950 50  0000 C CNN
+F 1 "Screw_Terminal_01x03" H 6850 4550 50  0000 C CNN
+F 2 "TerminalBlocks_Phoenix:TerminalBlock_Phoenix_MPT-2.54mm_3pol" H 6850 4750 50  0001 C CNN
+F 3 "" H 6850 4750 50  0001 C CNN
+	1    6850 4750
+	1    0    0    -1
+$EndComp
+$Comp
+L Conn_01x20 J6
+U 1 1 5B2BE603
+P 8550 4700
+F 0 "J6" H 8550 5700 50  0000 C CNN
+F 1 "Conn_01x20" H 8550 3600 50  0000 C CNN
+F 2 "Pin_Headers:Pin_Header_Straight_1x20_Pitch2.54mm" H 8550 4700 50  0001 C CNN
+F 3 "" H 8550 4700 50  0001 C CNN
+	1    8550 4700
+	1    0    0    -1
+$EndComp
+$Comp
+L Conn_01x07 J7
+U 1 1 5B2BF5F4
+P 4050 2550
+F 0 "J7" H 4050 2950 50  0000 C CNN
+F 1 "Conn_01x07" H 4050 2150 50  0000 C CNN
+F 2 "Pin_Headers:Pin_Header_Angled_1x07_Pitch2.54mm" H 4050 2550 50  0001 C CNN
+F 3 "" H 4050 2550 50  0001 C CNN
+	1    4050 2550
+	1    0    0    -1
+$EndComp
+$Comp
+L Screw_Terminal_01x02 J8
+U 1 1 5B2D3CFD
+P 2950 2400
+F 0 "J8" H 2950 2500 50  0000 C CNN
+F 1 "Screw_Terminal_01x02" H 2950 2200 50  0000 C CNN
+F 2 "TerminalBlocks_Phoenix:TerminalBlock_Phoenix_MPT-2.54mm_2pol" H 2950 2400 50  0001 C CNN
+F 3 "" H 2950 2400 50  0001 C CNN
+	1    2950 2400
+	1    0    0    -1
+$EndComp
+$Comp
+L Conn_01x04 J?
+U 1 1 5B2D3F13
+P 2100 2400
+F 0 "J?" H 2100 2600 50  0000 C CNN
+F 1 "Conn_01x04" H 2100 2100 50  0000 C CNN
+F 2 "" H 2100 2400 50  0001 C CNN
+F 3 "" H 2100 2400 50  0001 C CNN
+	1    2100 2400
+	1    0    0    -1
+$EndComp

Commit message: update
Parts:
- added C1, C2, C3, C4, C5, C6: C, Capacitors_SMD:C_0603, symbol C
- added C?: C, symbol C
- added D2: LED, LEDs:LED_0603, symbol LED
- added R3, R4, R5, R6, R7: R, Resistors_SMD:R_0603, symbol R
- added R? (x4): R, symbol R
- J9: renamed from J?; footprint (none) -> Pin_Headers:Pin_Header_Straight_1x04_Pitch2.54mm
- R1, R2: footprint Resistors_SMD:R_0805 -> Resistors_SMD:R_0603
Connections:
- no-connect marks 6 -> 7
Other:
- moved on the sheet: D1, J1, J2, J3, J4, J5, J6, J7, J8, J9, Q1, Q2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

Commit message: update
Parts:
- added J10: Micro_SD_Card, digikey-footprints:MicroSD_2908-05WB-MG, symbol Micro_SD_Card
- C7: renamed from C?; footprint (none) -> Capacitors_SMD:C_0603
- R10, R11, R8, R9: renamed from R?; footprint (none) -> Resistors_SMD:R_0603
Other:
- moved on the sheet: J2, J3, J4, J5, J6, Q1, Q2, R1, R10, R11, R2, R7
Changed lines of the file:
@@
 LIBS:switches
 LIBS:nqbit
+LIBS:RFM95
 LIBS:ESP32-wroover-adapter-cache
 EELAYER 25 0
@@
 L Q_NPN_BCE Q1
 U 1 1 5B2ADFF1
-P 4650 4100
-F 0 "Q1" H 4850 4150 50  0000 L CNN
-F 1 "Q_NPN_BCE" H 4850 4050 50  0000 L CNN
-F 2 "digikey-footprints:SOT-23-3" H 4850 4200 50  0001 C CNN
-F 3 "" H 4650 4100 50  0001 C CNN
-	1    4650 4100
+P 4200 3550
+F 0 "Q1" H 4400 3600 50  0000 L CNN
+F 1 "Q_NPN_BCE" H 4400 3500 50  0000 L CNN
+F 2 "digikey-footprints:SOT-23-3" H 4400 3650 50  0001 C CNN
+F 3 "" H 4200 3550 50  0001 C CNN
+	1    4200 3550
 	1    0    0    -1
 $EndComp
@@
 L Q_NPN_BCE Q2
 U 1 1 5B2AE090
-P 4650 4750
-F 0 "Q2" H 4850 4800 50  0000 L CNN
-F 1 "Q_NPN_BCE" H 4850 4700 50  0000 L CNN
-F 2 "digikey-footprints:SOT-23-3" H 4850 4850 50  0001 C CNN
-F 3 "" H 4650 4750 50  0001 C CNN
-	1    4650 4750
+P 4200 4200
+F 0 "Q2" H 4400 4250 50  0000 L CNN
+F 1 "Q_NPN_BCE" H 4400 4150 50  0000 L CNN
+F 2 "digikey-footprints:SOT-23-3" H 4400 4300 50  0001 C CNN
+F 3 "" H 4200 4200 50  0001 C CNN
+	1    4200 4200
 	1    0    0    -1
 $EndComp
@@
 L R R1
 U 1 1 5B2AE0EE
-P 4300 4100
-F 0 "R1" V 4380 4100 50  0000 C CNN
-F 1 "R" V 4300 4100 50  0000 C CNN
-F 2 "Resistors_SMD:R_0603" V 4230 4100 50  0001 C CNN
-F 3 "" H 4300 4100 50  0001 C CNN
-	1    4300 4100
+P 3850 3550
+F 0 "R1" V 3930 3550 50  0000 C CNN
+F 1 "R" V 3850 3550 50  0000 C CNN
+F 2 "Resistors_SMD:R_0603" V 3780 3550 50  0001 C CNN
+F 3 "" H 3850 3550 50  0001 C CNN
+	1    3850 3550
 	0    1    1    0
 $EndComp
@@
 L R R2
 U 1 1 5B2AE153
-P 4300 4750
-F 0 "R2" V 4380 4750 50  0000 C CNN
-F 1 "R" V 4300 4750 50  0000 C CNN
-F 2 "Resistors_SMD:R_0603" V 4230 4750 50  0001 C CNN
-F 3 "" H 4300 4750 50  0001 C CNN
-	1    4300 4750
+P 3850 4200
+F 0 "R2" V 3930 4200 50  0000 C CNN
+F 1 "R" V 3850 4200 50  0000 C CNN
+F 2 "Resistors_SMD:R_0603" V 3780 4200 50  0001 C CNN
+F 3 "" H 3850 4200 50  0001 C CNN
+	1    3850 4200
 	0    1    1    0
 $EndComp
@@
 L Screw_Terminal_01x03 J2
 U 1 1 5B2BE424
-P 6500 3700
-F 0 "J2" H 6500 3900 50  0000 C CNN
-F 1 "Screw_Terminal_01x03" H 6500 3500 50  0000 C CNN
-F 2 "TerminalBlocks_Phoenix:TerminalBlock_Phoenix_MPT-2.54mm_3pol" H 6500 3700 50  0001 C CNN
-F 3 "" H 6500 3700 50  0001 C CNN
-	1    6500 3700
+P 6050 3150
+F 0 "J2" H 6050 3350 50  0000 C CNN
+F 1 "Screw_Terminal_01x03" H 6050 2950 50  0000 C CNN
+F 2 "TerminalBlocks_Phoenix:TerminalBlock_Phoenix_MPT-2.54mm_3pol" H 6050 3150 50  0001 C CNN
+F 3 "" H 6050 3150 50  0001 C CNN
+	1    6050 3150
 	1    0    0    -1
 $EndComp
@@
 L Screw_Terminal_01x03 J3
 U 1 1 5B2BE4D6
-P 6500 4300
-F 0 "J3" H 6500 4500 50  0000 C CNN
-F 1 "Screw_Terminal_01x03" H 6500 4100 50  0000 C CNN
-F 2 "TerminalBlocks_Phoenix:TerminalBlock_Phoenix_MPT-2.54mm_3pol" H 6500 4300 50  0001 C CNN
-F 3 "" H 6500 4300 50  0001 C CNN
-	1    6500 4300
+P 6050 3750
+F 0 "J3" H 6050 3950 50  0000 C CNN
+F 1 "Screw_Terminal_01x03" H 6050 3550 50  0000 C CNN
+F 2 "TerminalBlocks_Phoenix:TerminalBlock_Phoenix_MPT-2.54mm_3pol" H 6050 3750 50  0001 C CNN
+F 3 "" H 6050 3750 50  0001 C CNN
+	1    6050 3750
 	1    0    0    -1
 $EndComp
@@
 L Screw_Terminal_01x03 J4
 U 1 1 5B2BE530
-P 6500 4850
-F 0 "J4" H 6500 5050 50  0000 C CNN
-F 1 "Screw_Terminal_01x03" H 6500 4650 50  0000 C CNN
-F 2 "TerminalBlocks_Phoenix:TerminalBlock_Phoenix_MPT-2.54mm_3pol" H 6500 4850 50  0001 C CNN
-F 3 "" H 6500 4850 50  0001 C CNN
-	1    6500 4850
+P 6050 4300
+F 0 "J4" H 6050 4500 50  0000 C CNN
+F 1 "Screw_Terminal_01x03" H 6050 4100 50  0000 C CNN
+F 2 "TerminalBlocks_Phoenix:TerminalBlock_Phoenix_MPT-2.54mm_3pol" H 6050 4300 50  0001 C CNN
+F 3 "" H 6050 4300 50  0001 C CNN
+	1    6050 4300
 	1    0    0    -1
 $EndComp
@@
 L Screw_Terminal_01x03 J5
 U 1 1 5B2BE57F
-P 6500 5650
-F 0 "J5" H 6500 5850 50  0000 C CNN
-F 1 "Screw_Terminal_01x03" H 6500 5450 50  0000 C CNN
-F 2 "TerminalBlocks_Phoenix:TerminalBlock_Phoenix_MPT-2.54mm_3pol" H 6500 5650 50  0001 C CNN
-F 3 "" H 6500 5650 50  0001 C CNN
-	1    6500 5650
+P 6050 5100
+F 0 "J5" H 6050 5300 50  0000 C CNN
+F 1 "Screw_Terminal_01x03" H 6050 4900 50  0000 C CNN
+F 2 "TerminalBlocks_Phoenix:TerminalBlock_Phoenix_MPT-2.54mm_3pol" H 6050 5100 50  0001 C CNN
+F 3 "" H 6050 5100 50  0001 C CNN
+	1    6050 5100
 	1    0    0    -1
 $EndComp
@@
 L Conn_01x20 J6
 U 1 1 5B2BE603
-P 9100 4650
-F 0 "J6" H 9100 5650 50  0000 C CNN
-F 1 "Conn_01x20" H 9100 3550 50  0000 C CNN
-F 2 "Pin_Headers:Pin_Header_Straight_1x20_Pitch2.54mm" H 9100 4650 50  0001 C CNN
-F 3 "" H 9100 4650 50  0001 C CNN
-	1    9100 4650
+P 8000 4550
+F 0 "J6" H 8000 5550 50  0000 C CNN
+F 1 "Conn_01x20" H 8000 3450 50  0000 C CNN
+F 2 "Pin_Headers:Pin_Header_Straight_1x20_Pitch2.54mm" H 8000 4550 50  0001 C CNN
+F 3 "" H 8000 4550 50  0001 C CNN
+	1    8000 4550
 	1    0    0    -1
 $EndComp
@@
 L R R7
 U 1 1 5B2D7BE3
-P 6850 3600
-F 0 "R7" V 6930 3600 50  0000 C CNN
-F 1 "R" V 6850 3600 50  0000 C CNN
-F 2 "Resistors_SMD:R_0603" V 6780 3600 50  0001 C CNN
-F 3 "" H 6850 3600 50  0001 C CNN
-	1    6850 3600
-	1    0    0    -1
-$EndComp
-$Comp
-L R R?
+P 6400 3050
+F 0 "R7" V 6480 3050 50  0000 C CNN
+F 1 "R" V 6400 3050 50  0000 C CNN
+F 2 "Resistors_SMD:R_0603" V 6330 3050 50  0001 C CNN
+F 3 "" H 6400 3050 50  0001 C CNN
+	1    6400 3050
+	1    0    0    -1
+$EndComp
+$Comp
+L R R11
 U 1 1 5B2D9E87
-P 5050 3400
-F 0 "R?" V 5130 3400 50  0000 C CNN
-F 1 "R" V 5050 3400 50  0000 C CNN
-F 2 "" V 4980 3400 50  0001 C CNN
-F 3 "" H 5050 3400 50  0001 C CNN
-	1    5050 3400
+P 4600 2850
+F 0 "R11" V 4680 2850 50  0000 C CNN
+F 1 "R" V 4600 2850 50  0000 C CNN
+F 2 "Resistors_SMD:R_0603" V 4530 2850 50  0001 C CNN
+F 3 "" H 4600 2850 50  0001 C CNN
+	1    4600 2850
 	-1   0    0    1
 $EndComp
 $Comp
-L R R?
+L R R10
 U 1 1 5B2D9F40
-P 5050 2950
-F 0 "R?" V 5130 2950 50  0000 C CNN
-F 1 "R" V 5050 2950 50  0000 C CNN
-F 2 "" V 4980 2950 50  0001 C CNN
-F 3 "" H 5050 2950 50  0001 C CNN
-	1    5050 2950
-	1    0    0    -1
-$EndComp
-$Comp
-L C C?
+P 4600 2400
+F 0 "R10" V 4680 2400 50  0000 C CNN
+F 1 "R" V 4600 2400 50  0000 C CNN
+F 2 "Resistors_SMD:R_0603" V 4530 2400 50  0001 C CNN
+F 3 "" H 4600 2400 50  0001 C CNN
+	1    4600 2400
+	1    0    0    -1
+$EndComp
+$Comp
+L C C7
 U 1 1 5B2DA485
 P 950 6650
-F 0 "C?" H 975 6750 50  0000 L CNN
+F 0 "C7" H 975 6750 50  0000 L CNN
 F 1 "C" H 975 6550 50  0000 L CNN
-F 2 "" H 988 6500 50  0001 C CNN
+F 2 "Capacitors_SMD:C_0603" H 988 6500 50  0001 C CNN
 F 3 "" H 950 6650 50  0001 C CNN
 	1    950  6650
@@
 $EndComp
 $Comp
-L R R?
+L R R8
 U 1 1 5B2DA9ED
 P 1600 6350
-F 0 "R?" V 1680 6350 50  0000 C CNN
+F 0 "R8" V 1680 6350 50  0000 C CNN
 F 1 "R" V 1600 6350 50  0000 C CNN
-F 2 "" V 1530 6350 50  0001 C CNN
+F 2 "Resistors_SMD:R_0603" V 1530 6350 50  0001 C CNN
 F 3 "" H 1600 6350 50  0001 C CNN
 	1    1600 6350
@@
 $EndComp
 $Comp
-L R R?
+L R R9
 U 1 1 5B2DAA68
 P 2000 6350
-F 0 "R?" V 2080 6350 50  0000 C CNN
+F 0 "R9" V 2080 6350 50  0000 C CNN
 F 1 "R" V 2000 6350 50  0000 C CNN
-F 2 "" V 1930 6350 50  0001 C CNN
+F 2 "Resistors_SMD:R_0603" V 1930 6350 50  0001 C CNN
 F 3 "" H 2000 6350 50  0001 C CNN
 	1    2000 6350
 	1    0    0    -1
 $EndComp
+$Comp
+L Micro_SD_Card J10
+U 1 1 5B2DAEB8
+P 10050 4100
+F 0 "J10" H 9400 4700 50  0000 C CNN
+F 1 "Micro_SD_Card" H 10700 4700 50  0000 R CNN
+F 2 "digikey-footprints:MicroSD_2908-05WB-MG" H 11200 4400 50  0001 C CNN
+F 3 "" H 10050 4100 50  0001 C CNN
+	1    10050 4100
+	1    0    0    -1
+$EndComp
